Commit message: add grip

File: urdf/reBot-DevArm_fixend_description/urdf/reBot-DevArm_fixend.urdf (robot description, URDF)
Before this commit: robot reBot-DevArm_fixend, 8 links, 7 joints
Joints:
- removed joint joint3
- added joint join3: type revolute, parent link2, child link3, origin xyz=-0.264 0 0 rpy=0 0 0, axis 0 0 1, limit lower=-3.14 upper=0 effort=27 velocity=50
- joint end_joint: origin xyz=-0.00018697 -5.9452E-05 0.14921 rpy=0 -1.5708 3.1415 -> xyz=0 0 0.15539 rpy=0 -1.5708 3.1415
- joint joint1: limit lower=-3.14 upper=3.14 effort=27 velocity=50 -> lower=-2.8 upper=2.8 effort=27 velocity=50; origin xyz=0 0 0.0708 rpy=0 0 0 -> xyz=-8.416E-05 0 0.08465 rpy=0 0 0
- joint joint2: origin xyz=0.02 0.035625 0.0497 rpy=-1.5708 0 0 -> xyz=0.020084 0.031625 0.05555 rpy=-1.5708 0 0
- joint joint4: origin xyz=0.2426 -0.054 -0.005625 rpy=0 0 0 -> xyz=0.2426 -0.054 -0.001625 rpy=0 0 0
- joint joint5: origin xyz=0.078308 -0.0355 -0.03 rpy=-1.5708 0 0 -> xyz=0.078308 -0.0375 -0.03 rpy=-1.5708 0 0
- joint joint6: limit lower=-6.28 upper=6.28 effort=7 velocity=200 -> lower=-3.14 upper=3.14 effort=7 velocity=200; origin xyz=0.027192 0 0.038 rpy=0 1.5708 0 -> xyz=0.028008 0 0.04 rpy=0 1.5708 0

Commit message: update G

File: urdf/reBot-DevArm_fixend_description/urdf/reBot-DevArm_fixend.urdf (robot description, URDF)
Before this commit: robot reBot-DevArm_fixend, 8 links, 7 joints
Links:
- link end_link: mass 0.25840000 -> 0.4000000
- link link4: mass 0.50800000 -> 0.52000000
- link link6: mass 0.34630000 -> 0.36630000
